Commit message: Fix right wheel joint axis (sim drove forward/turn swapped)
right_wheel_joint has rpy +pi/2, which turns its z axis to -y, so with
axis 0 0 1 a positive wheel speed rolled the robot backward. Forward made
the wheels fight (spin in place) and turning made them roll together.
Axis is now 0 0 -1 (like the Articulated Robotics template). Real robot
unaffected: diffdrive_arduino does not use the URDF axis.

Headless Gazebo check (room.world): 0.2 m/s x 3 s -> +0.529 m along x,
0.0 deg (odom 0.521 m); 0.5 rad/s x 3 s -> 0.000 m, +72.5 deg (odom +72.6).

Co-Authored-By: Claude Opus 5.5 <noreply@anthropic.com>

File: description/robot_core.xacro (robot description, xacro)
@@ -91,5 +91,6 @@
         <child link="right_wheel"/>
         <origin xyz="0 -0.175 0" rpy="${pi/2} 0 0"/>
-        <axis xyz="0 0 1"/>
+        <!-- Axis is -1 because rpy +pi/2 turns joint z to -y, so -z is +y and positive speed rolls forward like the left wheel -->
+        <axis xyz="0 0 -1"/>
         <dynamics damping="0.1" friction="0.1"/>
     </joint>
