Commit message: Add LiDAR launch from robot_ws, drive-test RViz config; fix rpy typos
- launch/lidar.launch.py + config/ldlidar.yaml: ldlidar_stl_ros2 from
  ~/robot_ws, frame laser_frame (URDF provides the TF), default /dev/ldlidar
- config/drive_test.rviz: fixed frame odom, robot model (transient local),
  /scan (best effort), TF
- lidar.xacro, camera.xacro: ryp= -> rpy= (camera optical rotation was ignored)
- package.xml: exec_depend ldlidar_stl_ros2; CLAUDE.md: drive-test procedure

Co-Authored-By: Claude Opus 5.5 <noreply@anthropic.com>

File: description/camera.xacro (robot description, xacro)
@@ -4,5 +4,5 @@
         <parent link="chassis"/>
         <child link="camera_link"/>
-        <origin xyz="0.305 0 0.08" ryp="0 0 0"/>
+        <origin xyz="0.305 0 0.08" rpy="0 0 0"/>
     </joint>
     <link name="camera_link">
@@ -17,5 +17,5 @@
         <parent link="camera_link"/>
         <child link="camera_link_optical"/>
-        <origin xyz="0 0 0" ryp="${-pi/2} 0 ${-pi/2}"/>
+        <origin xyz="0 0 0" rpy="${-pi/2} 0 ${-pi/2}"/>
     </joint>
     <link name="camera_link_optical"></link>

File: description/lidar.xacro (robot description, xacro)
@@ -4,5 +4,5 @@
         <parent link="chassis"/>
         <child link="laser_frame"/>
-        <origin xyz="0.175 0 0.175" ryp="0 0 0"/>
+        <origin xyz="0.175 0 0.175" rpy="0 0 0"/>
     </joint>
     <link name="laser_frame">
