Commit message: URDF: turtle drive, caster, lidar tower, 4-servo arm, phone mount
- description/weedbot_properties.xacro (all measurements, MEASURE markers), weedbot_body.xacro,
  weedbot_arm.xacro from ~/weedbot_urdf; robot.urdf.xacro includes them instead of robot_core,
  lidar, camera and phone_mount (files kept). base_link on the ground under the rear axle.
- Wheels = diff_cont values (r 0.06985, sep 0.1895); sim-only wheel override removed from
  gaz_ros2_ctl_use_sim.yaml; Gazebo wheel friction follows wheel_mu again.
- lidar_sim.xacro: Gazebo LD06 on laser_frame (min range 0.05, sees the tower column like the real one).
- Arm joints fixed in sim (no simulated servos: the arm collapsed into the scan plane).
- scripts/arm_joint_state_stub.py + config: arm (and real caster) joints at 0 on /joint_states,
  started by launch_robot and launch_sim.
- view_robot.launch.py + config/view_robot.rviz.
- Fix: robot_description passed as text (ParameterValue str) and rsp strips URDF comments. A
  "word: " in a comment broke YAML parsing, so launch_sim/launch_robot failed to start since
  3b156e3 (phone_mount.xacro) and gazebo_ros2_control could not load the wheel controllers.
- CLAUDE.md: Robot model section, sim test results, safety footprint/zones still to update.

Co-Authored-By: Claude Opus 5.5 <noreply@anthropic.com>

File: description/robot.urdf.xacro (robot description, xacro)
@@ -1,3 +1,8 @@
 <?xml version="1.0"?>
+<!-- WeedBot (rebuilt 2026-10): rear differential drive + front stem caster, lidar tower with the LD06
+     under the 4-servo arm, phone mount. All measurements: weedbot_properties.xacro (MEASURE markers).
+     base_link = on the ground under the centre of the rear axle.
+     Old files kept on disk but no longer included: robot_core.xacro, lidar.xacro, camera.xacro,
+     phone_mount.xacro (the body defines phone_mount -> phone_optical -> phone_link itself). -->
 <robot xmlns:xacro="http://www.ros.org/wiki/xacro"  name="robot">
     <xacro:arg name="use_ros2_control" default="true"/>
@@ -6,7 +11,12 @@
          e.g. 0.1 = slippery floor to show the EKF keeping the heading with the IMU. -->
     <xacro:arg name="wheel_mu" default="1.0"/>
-    <!-- Gazebo camera sensor (sim only). Off by default to save CPU; true for Phase 1 work. -->
+    <!-- Kept because rsp.launch.py passes it; unused since camera.xacro is no longer included
+         (the phone is the camera now). -->
     <xacro:arg name="sim_camera" default="false"/>
-    <xacro:include filename="robot_core.xacro" />
+    <!-- used by imu.xacro (was defined in the old robot_core.xacro) -->
+    <material name="blue"><color rgba="0.2 0.2 1 1"/></material>
+    <xacro:include filename="weedbot_properties.xacro"/>
+    <xacro:include filename="weedbot_body.xacro"/>
+    <xacro:include filename="weedbot_arm.xacro"/>
     <!--<xacro:include filename="gazebo_control.xacro"/>-->
     <xacro:if value="$(arg use_ros2_control)">
@@ -16,11 +26,9 @@
         <xacro:include filename="gazebo_control.xacro"/>
     </xacro:unless>
-    <xacro:include filename="lidar.xacro"/>
     <xacro:include filename="imu.xacro"/>
     <xacro:if value="$(arg sim_mode)">
         <xacro:include filename="imu_sim.xacro"/>
+        <xacro:include filename="lidar_sim.xacro"/>
         <xacro:include filename="sim_ground_truth.xacro"/>
     </xacro:if>
-    <xacro:include filename="camera.xacro"/>
-    <xacro:include filename="phone_mount.xacro"/>
 </robot>
