Commit message: Add sim/real switch, nav2 + SLAM configs, joystick and lawnmower script
Previously uncommitted work from the VM: sim_mode/use_ros2_control xacro
switch, measured wheel values, base_footprint link, nav2/slam_toolbox/
twist_mux/joystick configs and launch files, and scripts/lawnmower.py.

Co-Authored-By: Claude Opus 5.5 <noreply@anthropic.com>

File: description/gazebo_control.xacro (robot description, xacro)
@@ -6,6 +6,6 @@
             <left_joint>left_wheel_joint</left_joint>
             <right_joint>right_wheel_joint</right_joint>
-            <wheel_separation>0.35</wheel_separation>
-            <wheel_diameter>0.1</wheel_diameter>
+            <wheel_separation>0.22</wheel_separation>
+            <wheel_diameter>0.1397</wheel_diameter>
             <!-- Limits -->
             <max_wheel_torque>200</max_wheel_torque>

File: description/robot.urdf.xacro (robot description, xacro)
@@ -1,7 +1,13 @@
 <?xml version="1.0"?>
 <robot xmlns:xacro="http://www.ros.org/wiki/xacro"  name="robot">
+    <xacro:arg name="use_ros2_control" default="true"/>
     <xacro:include filename="robot_core.xacro" />
     <!--<xacro:include filename="gazebo_control.xacro"/>-->
-    <xacro:include filename="ros2_control.xacro"/>
+    <xacro:if value="$(arg use_ros2_control)">
+        <xacro:include filename="ros2_control.xacro"/>
+    </xacro:if>
+    <xacro:unless value="$(arg use_ros2_control)">
+        <xacro:include filename="gazebo_control.xacro"/>
+    </xacro:unless>
     <xacro:include filename="lidar.xacro"/>
     <xacro:include filename="camera.xacro"/>

File: description/robot_core.xacro (robot description, xacro)
@@ -18,4 +18,12 @@
     </material>
     <link name="base_link">
+    </link>
+     <!-- BASE_FOOTPRINT -->
+    <joint name="base_footprint_joint" type="fixed">
+        <parent link="base_link"/>
+        <child link="base_footprint"/>
+        <origin xyz="0 0 0" rpy="0 0 0"/>
+    </joint>
+    <link name="base_footprint">
     </link>
     <joint name="chassis_joint" type="fixed">

File: description/ros2_control.xacro (robot description, xacro)
@@ -1,56 +1,61 @@
 <?xml version="1.0"?>
 <robot xmlns:xacro="http://www.ros.org/wiki/xacro">
-    <ros2_control name="RealRobot" type="system">
-        <hardware>
-            <plugin>diffdrive_arduino/DiffDriveArduinoHardware</plugin>
-            <param name="left_wheel_name">left_wheel_joint</param>
-            <param name="right_wheel_name">right_wheel_joint</param>
-            <param name="loop_rate">10</param>
-            <param name="device">/dev/ttyUSB0</param>
-            <param name="baud_rate">57600</param>
-            <param name="timeout_ms">2000</param>
-            <param name="enc_counts_per_rev">1980</param>
-        </hardware>
-        <joint name="left_wheel_joint">
-            <command_interface name="velocity">
-                <param name="min">-10</param>
-                <param name="max">10</param>
-            </command_interface>
-            <state_interface name="position"/>
-            <state_interface name="velocity"/>
-        </joint>
-        <joint name="right_wheel_joint">
-            <command_interface name="velocity">
-                <param name="min">-10</param>
-                <param name="max">10</param>
-            </command_interface>
-            <state_interface name="position"/>
-            <state_interface name="velocity"/>
-        </joint>
-    </ros2_control>
-    <!-- <ros2_control name="GazeboSystem" type="system">
-        <hardware>
-            <plugin>gazebo_ros2_control/GazeboSystem</plugin>
-        </hardware>
-        <joint name="left_wheel_joint">
-            <command_interface name="velocity">
-                <param name="min">-10</param>
-                <param name="max">10</param>
-            </command_interface>
-            <state_interface name="velocity"/>
-            <state_interface name="position"/>
-        </joint>
-        <joint name="right_wheel_joint">
-            <command_interface name="velocity">
-                <param name="min">-10</param>
-                <param name="max">10</param>
-            </command_interface>
-            <state_interface name="velocity"/>
-            <state_interface name="position"/>
-        </joint>
-    </ros2_control> -->
+    <xacro:unless value="$(arg sim_mode)">
+        <ros2_control name="RealRobot" type="system">
+            <hardware>
+                <plugin>diffdrive_arduino/DiffDriveArduinoHardware</plugin>
+                <param name="left_wheel_name">left_wheel_joint</param>
+                <param name="right_wheel_name">right_wheel_joint</param>
+                <param name="loop_rate">10</param>
+                <param name="device">/dev/ttyUSB1</param>
+                <param name="baud_rate">57600</param>
+                <param name="timeout_ms">2000</param>
+                <param name="enc_counts_per_rev">3436</param>
+            </hardware>
+            <joint name="left_wheel_joint">
+                <command_interface name="velocity">
+                    <param name="min">-10</param>
+                    <param name="max">10</param>
+                </command_interface>
+                <state_interface name="position"/>
+                <state_interface name="velocity"/>
+            </joint>
+            <joint name="right_wheel_joint">
+                <command_interface name="velocity">
+                    <param name="min">-10</param>
+                    <param name="max">10</param>
+                </command_interface>
+                <state_interface name="position"/>
+                <state_interface name="velocity"/>
+            </joint>
+        </ros2_control>
+    </xacro:unless>
+    <xacro:if value="$(arg sim_mode)">
+        <ros2_control name="GazeboSystem" type="system">
+            <hardware>
+                <plugin>gazebo_ros2_control/GazeboSystem</plugin>
+            </hardware>
+            <joint name="left_wheel_joint">
+                <command_interface name="velocity">
+                    <param name="min">-10</param>
+                    <param name="max">10</param>
+                </command_interface>
+                <state_interface name="velocity"/>
+                <state_interface name="position"/>
+            </joint>
+            <joint name="right_wheel_joint">
+                <command_interface name="velocity">
+                    <param name="min">-10</param>
+                    <param name="max">10</param>
+                </command_interface>
+                <state_interface name="velocity"/>
+                <state_interface name="position"/>
+            </joint>
+        </ros2_control>
+    </xacro:if>
     <gazebo>
         <plugin name="gazebo_ros2_control" filename="libgazebo_ros2_control.so">
             <parameters>$(find my_bot)/config/my_controllers.yaml</parameters>
+            <parameters>$(find my_bot)/config/gaz_ros2_ctl_use_sim.yaml</parameters>
         </plugin>
     </gazebo>

Commit message: URDF: real v17 measurements, rear lidar tower, spray tank, footprint
- weedbot_properties.xacro: CAD "project 101 v17" values (wheels r 0.0635 / sep 0.176, frame,
  caster at the nose x 0.419, rear lidar tower, arm lengths, phone camera 0.0498 left of centre)
  plus top frame, body shell, spray tank + sump (3.6 kg) and wrist roll
- weedbot_body.xacro: top frame + cover, body_shell, spray_tank, caster bracket, tower on the top
  cover with the column in front of the LD06 (laser_frame -0.036, 0, 0.268), cheeks at +-0.0235
- weedbot_arm.xacro: wrist_roll joint (0.0737 along the last link) -> nozzle -> spray_tip, yaw servo
  under the plate 0.0224 behind the axis; differently coloured parts in their own links (RViz draws
  all visuals of a link in the first one's colour)
- wheel values in my_controllers.yaml and gazebo_control.xacro match the URDF
- Nav2 footprint (8 points, robot_radius off) in both costmaps; safety.yaml zones and the
  scan_self_filter box (x -0.11..0.53, y +-0.16) for the new outline; self-hits now NaN, not +inf
  (inf_is_valid cleared the costmap through the tank's shadow)
- stub publishes wrist_roll; CLAUDE.md: heights, footprint, sim results and the BLIND-AHEAD warning
  (the tank hides +-27 deg straight ahead from the LiDAR)

Co-Authored-By: Claude Opus 5.5 <noreply@anthropic.com>

File: description/gazebo_control.xacro (robot description, xacro)
@@ -6,6 +6,6 @@
             <left_joint>left_wheel_joint</left_joint>
             <right_joint>right_wheel_joint</right_joint>
-            <wheel_separation>0.22</wheel_separation>
-            <wheel_diameter>0.1397</wheel_diameter>
+            <wheel_separation>${wheel_separation}</wheel_separation>
+            <wheel_diameter>${2*wheel_radius}</wheel_diameter>
             <!-- Limits -->
             <max_wheel_torque>200</max_wheel_torque>

File: description/lidar_sim.xacro (robot description, xacro)
@@ -21,6 +21,6 @@
         <range>
           <!-- 0.05: just outside the LD06 housing (radius 0.019), so the sim sees the tower column
-               0.06-0.10 m behind the laser like the real LD06 does (scan_self_filter removes it).
-               The old 0.12 was for the old 0.05 m housing and hid the column. -->
+               0.06-0.10 m in front of the laser and the spray tank like the real LD06 does
+               (scan_self_filter removes both). The old 0.12 was for the old 0.05 m housing. -->
           <min>0.05</min>
           <max>12</max>

File: description/weedbot_arm.xacro (robot description, xacro)
@@ -1,12 +1,15 @@
 <?xml version="1.0"?>
 <!--
-  4-servo sprayer arm (MG996R x4) on top of the lidar tower.
-    arm_base_yaw   : servo 1, turns the whole arm about the vertical axis (above the lidar)
+  Sprayer arm on top of the lidar tower (rear top of the robot): 4 x MG996R + a wrist roll.
+    arm_base_yaw   : servo 1, hangs under the base plate behind the axis and turns the arm through
+                     a gear, about the vertical axis above the lidar (yaw range: MEASURE)
     shoulder_pitch : servo 2
     elbow_pitch    : servo 3
-    wrist_pitch    : servo 4, carries the sprayer nozzle (link spray_tip = where the spray leaves)
-  Zero position = arm pointing straight up, folded over the robot. Positive pitch tilts forward.
-  Each joint: -90..+90 deg (the servo's 180 deg travel centred). Change arm_l1..l4 in
-  weedbot_properties.xacro to your real link lengths (axis to axis).
+    wrist_pitch    : servo 4
+    wrist_roll     : servo 5, wrist_roll_z along the last link, turns the nozzle about the link
+                     (link spray_tip = where the spray leaves)
+  Zero position = arm pointing straight up. Positive pitch tilts forward.
+  Each joint: -90..+90 deg (the servo's 180 deg travel centred). Link lengths (axis to axis) are in
+  weedbot_properties.xacro (arm_l1..l4, wrist_roll_z, CAD v17). Masses: MEASURE.
   In RViz, move it with joint_state_publisher_gui; on the robot the servo driver publishes the same
   joint names on /joint_states.
@@ -15,5 +18,5 @@
   <!-- Gazebo has no servos for the arm yet: with revolute joints the arm collapsed under gravity
        (forearm hanging through the LiDAR scan plane) while TF still showed it straight up. In sim
-       the four joints are fixed at 0 (= what arm_joint_state_stub.py reports); on the robot they are
+       the five joints are fixed at 0 (= what arm_joint_state_stub.py reports); on the robot they are
        servo joints. Give them a simulated position controller before moving the arm in sim. -->
   <xacro:if value="$(arg sim_mode)"><xacro:property name="arm_joint_type" value="fixed"/></xacro:if>
@@ -48,5 +51,5 @@
     </link>
   </xacro:macro>
-  <!-- base plate on the tower, directly above the lidar -->
+  <!-- base plate on the tower, directly above the lidar; the yaw servo hangs under it -->
   <joint name="arm_base_joint" type="fixed">
     <parent link="base_link"/>
@@ -56,9 +59,17 @@
   <link name="arm_base">
     <visual><geometry><cylinder radius="${arm_plate_r}" length="${arm_plate_t}"/></geometry><material name="petg_blue"/></visual>
-    <!-- the plate reaches back to the column -->
-    <visual><origin xyz="${(tower_x-arm_x)/2} 0 0"/><geometry><box size="${arm_x-tower_x} ${tower_w+0.02} ${arm_plate_t}"/></geometry><material name="petg_blue"/></visual>
+    <!-- the plate reaches forward to the column -->
+    <visual><origin xyz="${(tower_x-arm_x)/2} 0 0"/><geometry><box size="${fabs(arm_x-tower_x)} ${tower_w+0.02} ${arm_plate_t}"/></geometry><material name="petg_blue"/></visual>
     <collision><geometry><cylinder radius="${arm_plate_r}" length="${arm_plate_t}"/></geometry></collision>
     <inertial><mass value="0.15"/><xacro:cyl_inertia m="0.15" r="${arm_plate_r}" h="${arm_plate_t}"/></inertial>
   </link>
+  <!-- yaw servo (servo 1) under the plate, arm_yaw_servo_dx behind the axis, shaft up into the gear
+       (drawn as a full MG996R box hanging from the plate: check the clearance to the LD06 in CAD) -->
+  <joint name="arm_yaw_servo_joint" type="fixed">
+    <parent link="arm_base"/>
+    <child link="arm_yaw_servo"/>
+    <origin xyz="${arm_yaw_servo_dx} 0 ${-arm_plate_t/2-servo_z/2}"/>
+  </joint>
+  <link name="arm_yaw_servo"><xacro:servo_visual xyz="0 0 0" rpy="0 0 0"/></link>
   <!-- servo 1: yaw -->
   <joint name="arm_base_yaw" type="${arm_joint_type}">
@@ -70,9 +81,12 @@
   </joint>
   <link name="arm_turret">
-    <!-- servo 1 body sits under the plate inside the tower cut-out; the turret disc on top -->
+    <visual><origin xyz="0 0 ${arm_l1/2}"/><geometry><box size="${link_w} ${link_w} ${arm_l1}"/></geometry><material name="petg_blue"/></visual>
+    <inertial><origin xyz="0 0 ${arm_l1/2}"/><mass value="0.09"/><xacro:box_inertia m="0.09" x="${servo_x}" y="${servo_y}" z="${arm_l1}"/></inertial>
+  </link>
+  <!-- turret disc on the plate and servo 2 (shoulder) body at the top -->
+  <joint name="turret_servo_joint" type="fixed"><parent link="arm_turret"/><child link="turret_servo"/><origin xyz="0 0 0"/></joint>
+  <link name="turret_servo">
     <visual><origin xyz="0 0 0.004"/><geometry><cylinder radius="0.030" length="0.008"/></geometry><material name="servo"/></visual>
     <xacro:servo_visual xyz="0 0 ${arm_l1-servo_z/2+0.005}" rpy="0 0 0"/>
-    <visual><origin xyz="0 0 ${arm_l1/2}"/><geometry><box size="${link_w} ${link_w} ${arm_l1}"/></geometry><material name="petg_blue"/></visual>
-    <inertial><origin xyz="0 0 ${arm_l1/2}"/><mass value="0.09"/><xacro:box_inertia m="0.09" x="${servo_x}" y="${servo_y}" z="${arm_l1}"/></inertial>
   </link>
   <!-- servo 2: shoulder -->
@@ -94,5 +108,5 @@
   </joint>
   <xacro:arm_link name="forearm" length="${arm_l3}" mass="0.07"/>
-  <!-- servo 4: wrist, carries the nozzle -->
+  <!-- servo 4: wrist pitch -->
   <joint name="wrist_pitch" type="${arm_joint_type}">
     <parent link="forearm"/>
@@ -103,14 +117,33 @@
   </joint>
   <link name="wrist">
+    <visual><origin xyz="0 0 ${wrist_roll_z/2}"/><geometry><box size="${link_w} ${link_w} ${wrist_roll_z}"/></geometry><material name="petg_blue"/></visual>
+    <collision><origin xyz="0 0 ${wrist_roll_z/2}"/><geometry><box size="${servo_x} ${servo_y} ${wrist_roll_z+servo_z}"/></geometry></collision>
+    <inertial><origin xyz="0 0 ${wrist_roll_z/2}"/><mass value="0.1"/><xacro:box_inertia m="0.1" x="${servo_x}" y="${servo_y}" z="${wrist_roll_z}"/></inertial>
+  </link>
+  <!-- servo 4 body at the wrist pitch axis and servo 5 (wrist roll) body, shaft along the link at the
+       roll joint (size approximate), visual only -->
+  <joint name="wrist_servos_joint" type="fixed"><parent link="wrist"/><child link="wrist_servos"/><origin xyz="0 0 0"/></joint>
+  <link name="wrist_servos">
     <xacro:servo_visual xyz="0 0 0" rpy="0 0 0"/>
-    <visual><origin xyz="0 0 ${arm_l4/2}"/><geometry><cylinder radius="0.006" length="${arm_l4}"/></geometry><material name="alu"/></visual>
-    <collision><origin xyz="0 0 ${arm_l4/2}"/><geometry><box size="${servo_x} ${servo_y} ${arm_l4+servo_z}"/></geometry></collision>
-    <inertial><origin xyz="0 0 ${arm_l4/2}"/><mass value="0.08"/><xacro:box_inertia m="0.08" x="${servo_x}" y="${servo_y}" z="${arm_l4}"/></inertial>
+    <visual><origin xyz="0 0 ${wrist_roll_z-servo_x/2}"/><geometry><box size="${servo_y} ${servo_z} ${servo_x}"/></geometry><material name="servo"/></visual>
+  </link>
+  <!-- servo 5: wrist roll, turns the nozzle about the link axis -->
+  <joint name="wrist_roll" type="${arm_joint_type}">
+    <parent link="wrist"/>
+    <child link="nozzle"/>
+    <origin xyz="0 0 ${wrist_roll_z}"/>
+    <axis xyz="0 0 1"/>
+    <limit lower="${-servo_limit}" upper="${servo_limit}" effort="${servo_effort}" velocity="${servo_velocity}"/>
+  </joint>
+  <link name="nozzle">
+    <visual><origin xyz="0 0 ${(arm_l4-wrist_roll_z)/2}"/><geometry><cylinder radius="0.006" length="${arm_l4-wrist_roll_z}"/></geometry><material name="alu"/></visual>
+    <collision><origin xyz="0 0 ${(arm_l4-wrist_roll_z)/2}"/><geometry><cylinder radius="0.006" length="${arm_l4-wrist_roll_z}"/></geometry></collision>
+    <inertial><origin xyz="0 0 ${(arm_l4-wrist_roll_z)/2}"/><mass value="0.02"/><xacro:cyl_inertia m="0.02" r="0.006" h="${arm_l4-wrist_roll_z}"/></inertial>
   </link>
   <!-- where the spray comes out, z pointing along the nozzle -->
   <joint name="spray_tip_joint" type="fixed">
-    <parent link="wrist"/>
+    <parent link="nozzle"/>
     <child link="spray_tip"/>
-    <origin xyz="0 0 ${arm_l4}"/>
+    <origin xyz="0 0 ${arm_l4-wrist_roll_z}"/>
   </joint>
   <link name="spray_tip">
