Commit message: URDF: v19 arm on the body, LD06 on the tank
- lidar tower and lidar_shelf removed; arm base set into the top cover (arm_x -0.0066,
  arm_base_z 0.2305, arm_plate_t 0.0061 -> yaw joint 0.2366)
- LD06 on a 50 x 50 x 8 mm puck on the spray tank: lidar_x 0.2495, lidar_base_z 0.3554,
  scan plane 0.3784 (above the tank: the front is visible again; the arm blocks ~32 deg behind)
- sim LiDAR min range 0.05 -> 0.14: rays starting above the tank top gave flickering false
  Gazebo hits at the tank's rear edge (0.052 m)
- comments in safety.yaml, nav2_params.yaml, scan_self_filter.py; CLAUDE.md: v19 heights,
  sim results, LiDAR limits (nothing below 0.378 m, rear blind behind the arm)

Co-Authored-By: Claude Opus 5.5 <noreply@anthropic.com>

File: description/lidar_sim.xacro (robot description, xacro)
@@ -20,8 +20,11 @@
         </scan>
         <range>
-          <!-- 0.05: just outside the LD06 housing (radius 0.019), so the sim sees the tower column
-               0.06-0.10 m in front of the laser and the spray tank like the real LD06 does
-               (scan_self_filter removes both). The old 0.12 was for the old 0.05 m housing. -->
-          <min>0.05</min>
+          <!-- 0.14 (v19, LD06 on the tank): every ray must START outside the tank's outline seen from
+               above (farthest tank corner 0.130 m from the laser). With 0.05 the backward rays started
+               above the tank top (2.4 cm below the scan plane) and Gazebo's ray-box test reported
+               flickering false hits at the tank's rear edge (0.052 m) whenever the robot pitched a
+               hair nose-up. Everything within 0.14 m is inside scan_self_filter's box anyway. The arm
+               (0.256 m behind) still shows up like on the real LD06 (min range 0.02). -->
+          <min>0.14</min>
           <max>12</max>
           <resolution>0.01</resolution>

File: description/robot.urdf.xacro (robot description, xacro)
@@ -1,5 +1,5 @@
 <?xml version="1.0"?>
-<!-- WeedBot (rebuilt 2026-10): rear differential drive + front stem caster, lidar tower with the LD06
-     under the 4-servo arm, phone mount. All measurements: weedbot_properties.xacro (MEASURE markers).
+<!-- WeedBot (rebuilt 2026-10): rear differential drive + front stem caster, spray tank with the LD06
+     on top, sprayer arm on the top cover, phone mount. All measurements: weedbot_properties.xacro (MEASURE markers).
      base_link = on the ground under the centre of the rear axle.
      Old files kept on disk but no longer included: robot_core.xacro, lidar.xacro, camera.xacro,

File: description/weedbot_arm.xacro (robot description, xacro)
@@ -1,7 +1,7 @@
 <?xml version="1.0"?>
 <!--
-  Sprayer arm on top of the lidar tower (rear top of the robot): 4 x MG996R + a wrist roll.
+  Sprayer arm on the top cover (rear of the robot, CAD v19): 4 x MG996R + a wrist roll.
     arm_base_yaw   : servo 1, hangs under the base plate behind the axis and turns the arm through
-                     a gear, about the vertical axis above the lidar (yaw range: MEASURE)
+                     a gear, about the vertical axis at arm_x (yaw range: MEASURE)
     shoulder_pitch : servo 2
     elbow_pitch    : servo 3
@@ -51,5 +51,5 @@
     </link>
   </xacro:macro>
-  <!-- base plate on the tower, directly above the lidar; the yaw servo hangs under it -->
+  <!-- base plate set into the top cover (top = cover top = yaw joint); the yaw servo hangs under it -->
   <joint name="arm_base_joint" type="fixed">
     <parent link="base_link"/>
@@ -59,11 +59,9 @@
   <link name="arm_base">
     <visual><geometry><cylinder radius="${arm_plate_r}" length="${arm_plate_t}"/></geometry><material name="petg_blue"/></visual>
-    <!-- the plate reaches forward to the column -->
-    <visual><origin xyz="${(tower_x-arm_x)/2} 0 0"/><geometry><box size="${fabs(arm_x-tower_x)} ${tower_w+0.02} ${arm_plate_t}"/></geometry><material name="petg_blue"/></visual>
     <collision><geometry><cylinder radius="${arm_plate_r}" length="${arm_plate_t}"/></geometry></collision>
     <inertial><mass value="0.15"/><xacro:cyl_inertia m="0.15" r="${arm_plate_r}" h="${arm_plate_t}"/></inertial>
   </link>
-  <!-- yaw servo (servo 1) under the plate, arm_yaw_servo_dx behind the axis, shaft up into the gear
-       (drawn as a full MG996R box hanging from the plate: check the clearance to the LD06 in CAD) -->
+  <!-- yaw servo (servo 1) under the plate (inside the body), arm_yaw_servo_dx behind the axis, shaft
+       up into the gear -->
   <joint name="arm_yaw_servo_joint" type="fixed">
     <parent link="arm_base"/>

File: description/weedbot_body.xacro (robot description, xacro)
@@ -2,6 +2,7 @@
 <!--
   WeedBot body: bottom + top frame, body shell, rear drive wheels, front stem caster (the nose),
-  electronics plate, spray tank, lidar tower with the LD06 at the rear top under the arm base, and
-  the phone mount. Include from robot.urdf.xacro:
+  electronics plate, spray tank with the LD06 on top (on a puck), and the phone mount. The arm base
+  sits on the top cover (weedbot_arm.xacro); there is no lidar tower since CAD v19.
+  Include from robot.urdf.xacro:
       <xacro:include filename="weedbot_properties.xacro"/>
       <xacro:include filename="weedbot_body.xacro"/>
@@ -260,25 +261,15 @@
     </link>
   </xacro:unless>
-  <!-- =============================== lidar tower + LD06 =============================== -->
-  <!-- one column at the rear top, standing on the top cover; the LD06 sits on a shelf BEHIND it and
-       the arm base plate on top. In the scan plane: the column (inside the tank's shadow) and the
-       spray tank = ~54 deg blind sector straight ahead (removed by scan_self_filter). -->
-  <joint name="tower_joint" type="fixed">
-    <parent link="base_link"/>
-    <child link="tower"/>
-    <origin xyz="${tower_x} 0 ${(tower_base_z+arm_base_z)/2}"/>
-  </joint>
-  <link name="tower">
-    <visual><geometry><box size="${tower_d} ${tower_w} ${arm_base_z-tower_base_z}"/></geometry><material name="petg_blue"/></visual>
-    <collision><geometry><box size="${tower_d} ${tower_w} ${arm_base_z-tower_base_z}"/></geometry></collision>
-    <inertial><mass value="0.2"/><xacro:box_inertia m="0.2" x="${tower_d}" y="${tower_w}" z="${arm_base_z-tower_base_z}"/></inertial>
-  </link>
-  <joint name="lidar_shelf_joint" type="fixed">
-    <parent link="base_link"/>
-    <child link="lidar_shelf"/>
-    <origin xyz="${(tower_x+lidar_x)/2} 0 ${lidar_base_z-shelf_t/2}"/>
-  </joint>
-  <link name="lidar_shelf">
-    <visual><geometry><box size="${fabs(lidar_x-tower_x)+lidar_dia} ${lidar_dia+0.02} ${shelf_t}"/></geometry><material name="petg_blue"/></visual>
+  <!-- =============================== LD06 on the spray tank =============================== -->
+  <!-- puck on the tank top, LD06 on the puck. In the scan plane (0.378) only the arm: ~32 deg blind
+       sector straight behind (removed by scan_self_filter). -->
+  <joint name="lidar_puck_joint" type="fixed">
+    <parent link="base_link"/>
+    <child link="lidar_puck"/>
+    <origin xyz="${lidar_x} 0 ${puck_z0+puck_h/2}"/>
+  </joint>
+  <link name="lidar_puck">
+    <visual><geometry><box size="${puck_size} ${puck_size} ${puck_h}"/></geometry><material name="petg_blue"/></visual>
+    <collision><geometry><box size="${puck_size} ${puck_size} ${puck_h}"/></geometry></collision>
   </link>
   <joint name="lidar_joint" type="fixed">

File: description/weedbot_properties.xacro (robot description, xacro)
@@ -1,8 +1,8 @@
 <?xml version="1.0"?>
 <!--
-  ONE place for every measurement of the real WeedBot. Everything else (body, arm, lidar tower,
+  ONE place for every measurement of the real WeedBot. Everything else (body, arm, LD06,
   phone mount, Gazebo) reads from here. Units: metres and radians. Frame: x forward, y left, z up.
   base_link = on the GROUND, under the centre of the rear (drive) axle.
-  Source: FreeCAD "project 101 v17" (2026-10-18). Values still marked MEASURE are estimates
+  Source: FreeCAD "project 101 v17" (2026-10-18), arm base and LD06 moved per v19. Values still marked MEASURE are estimates
   (IMU position in imu.xacro, masses other than the tank, caster trail, arm yaw range).
 -->
@@ -46,19 +46,17 @@
   <!-- printed gear cheeks beside the axle gears (visual only) -->
   <xacro:property name="cheek_y" value="0.0235"/>
-  <!-- lidar tower at the REAR TOP, standing on the top cover. The LD06 sits on a shelf on the BACK of
-       the column (column in front of the lidar), under the arm base plate. -->
-  <xacro:property name="tower_x"        value="0.0436"/>    <!-- column centre, in front of the lidar -->
-  <xacro:property name="tower_w"        value="0.020"/>     <!-- column width (y) -->
-  <xacro:property name="tower_d"        value="0.040"/>     <!-- column depth (x) -->
-  <xacro:property name="tower_base_z"   value="0.2366"/>    <!-- column foot = top cover -->
-  <xacro:property name="lidar_x"        value="-0.0364"/>   <!-- LD06 centre -->
-  <xacro:property name="lidar_base_z"   value="0.2446"/>    <!-- bottom of the LD06; scan plane = base + lidar_scan_dz = 0.2676 -->
+  <!-- LD06 on top of the spray tank (v19; no lidar tower any more), on a puck. The scan plane is
+       above everything except the arm: ~32 deg blind sector straight behind (the arm). -->
+  <xacro:property name="lidar_x"        value="0.2495"/>    <!-- LD06 centre -->
+  <xacro:property name="lidar_base_z"   value="0.3554"/>    <!-- bottom of the LD06; scan plane = base + lidar_scan_dz = 0.3784 -->
   <xacro:property name="lidar_dia"      value="0.0386"/>
   <xacro:property name="lidar_h"        value="0.035"/>
   <xacro:property name="lidar_scan_dz"  value="0.023"/>     <!-- LD06 optical centre above its bottom face -->
   <xacro:property name="lidar_frame"    value="laser_frame"/>   <!-- must match the ldlidar driver frame_id -->
-  <xacro:property name="shelf_t"        value="0.005"/>
+  <xacro:property name="puck_size"      value="0.050"/>     <!-- square puck under the LD06, on the tank top -->
+  <xacro:property name="puck_h"         value="0.008"/>
+  <xacro:property name="puck_z0"        value="0.3474"/>    <!-- puck bottom; puck top = LD06 bottom -->
   <!-- spray tank on the top frame at the front, with a sump below it (top of the sump = tank_z0).
-       It is in the LiDAR scan plane: ~54 deg blind sector straight ahead. -->
+       Carries the LD06 (below the scan plane since v19). -->
   <xacro:property name="tank_x0"   value="0.198"/>
   <xacro:property name="tank_x1"   value="0.294"/>
@@ -72,7 +70,7 @@
   <xacro:property name="tank_mass" value="3.6"/>
   <!-- robotic arm: 4 x MG996R pitch/yaw (40.7 x 19.7 x 42.9 mm, 180 deg) + wrist roll -->
-  <xacro:property name="arm_x"          value="${lidar_x}"/>   <!-- base yaw axis directly above the lidar -->
-  <xacro:property name="arm_base_z"     value="0.3136"/>     <!-- underside of the arm base plate -->
-  <xacro:property name="arm_plate_t"    value="0.006"/>
+  <xacro:property name="arm_x"          value="-0.0066"/>    <!-- base yaw axis (v19: arm base on the top cover) -->
+  <xacro:property name="arm_base_z"     value="0.2305"/>     <!-- underside of the arm base plate (= top of the top frame) -->
+  <xacro:property name="arm_plate_t"    value="0.0061"/>     <!-- plate top = yaw joint = top of the cover, 0.2366 -->
   <xacro:property name="arm_plate_r"    value="0.060"/>
   <xacro:property name="arm_yaw_servo_dx" value="-0.0224"/>  <!-- yaw servo under the plate, behind the axis (drives a gear) -->

Commit message: URDF: v19 CAD numbers, parked arm pose, tank top 0.3474
- tank top 0.3474 (= puck bottom; filler cap to 0.3604 not modelled), arm_l1 0.07065
- arm parked as in CAD v19 (elbow +90 deg, wrist +90 deg: forearm forward, nozzle down at
  x 0.0934, z 0.27625): fixed in that pose in sim, published by arm_joint_state_stub.yaml,
  view_robot sliders start there
- wrist collision box widened to the CAD scan envelope (arm_scan_w 0.078): sim now shows the
  real ~32 deg blind sector behind the LD06
- CLAUDE.md: v19 heights, parked pose, sim results

Co-Authored-By: Claude Opus 5.5 <noreply@anthropic.com>

File: description/lidar_sim.xacro (robot description, xacro)
@@ -24,6 +24,7 @@
                above the tank top (2.4 cm below the scan plane) and Gazebo's ray-box test reported
                flickering false hits at the tank's rear edge (0.052 m) whenever the robot pitched a
-               hair nose-up. Everything within 0.14 m is inside scan_self_filter's box anyway. The arm
-               (0.256 m behind) still shows up like on the real LD06 (min range 0.02). -->
+               hair nose-up. Everything within 0.14 m is inside scan_self_filter's box anyway. The
+               parked arm still gives the real ~32 deg sector behind; its wrist's near face (0.136 m)
+               is just inside 0.14, so the sim reports the far face (0.176 m): filtered either way. -->
           <min>0.14</min>
           <max>12</max>

File: description/weedbot_arm.xacro (robot description, xacro)
@@ -18,8 +18,23 @@
   <!-- Gazebo has no servos for the arm yet: with revolute joints the arm collapsed under gravity
        (forearm hanging through the LiDAR scan plane) while TF still showed it straight up. In sim
-       the five joints are fixed at 0 (= what arm_joint_state_stub.py reports); on the robot they are
-       servo joints. Give them a simulated position controller before moving the arm in sim. -->
-  <xacro:if value="$(arg sim_mode)"><xacro:property name="arm_joint_type" value="fixed"/></xacro:if>
-  <xacro:unless value="$(arg sim_mode)"><xacro:property name="arm_joint_type" value="revolute"/></xacro:unless>
+       the five joints are FIXED in the parked pose (arm_park_*, the joint origins carry the angles;
+       = what arm_joint_state_stub.py reports on the robot); on the robot they are servo joints at 0
+       in the origins. Give them a simulated position controller before moving the arm in sim. -->
+  <xacro:if value="$(arg sim_mode)">
+    <xacro:property name="arm_joint_type" value="fixed"/>
+    <xacro:property name="q_yaw" value="${arm_park_yaw}"/>
+    <xacro:property name="q_shoulder" value="${arm_park_shoulder}"/>
+    <xacro:property name="q_elbow" value="${arm_park_elbow}"/>
+    <xacro:property name="q_wrist" value="${arm_park_wrist}"/>
+    <xacro:property name="q_roll" value="${arm_park_roll}"/>
+  </xacro:if>
+  <xacro:unless value="$(arg sim_mode)">
+    <xacro:property name="arm_joint_type" value="revolute"/>
+    <xacro:property name="q_yaw" value="0"/>
+    <xacro:property name="q_shoulder" value="0"/>
+    <xacro:property name="q_elbow" value="0"/>
+    <xacro:property name="q_wrist" value="0"/>
+    <xacro:property name="q_roll" value="0"/>
+  </xacro:unless>
   <xacro:property name="servo_x" value="0.0407"/>
   <xacro:property name="servo_y" value="0.0197"/>
@@ -74,5 +89,5 @@
     <parent link="arm_base"/>
     <child link="arm_turret"/>
-    <origin xyz="0 0 ${arm_plate_t/2}"/>
+    <origin xyz="0 0 ${arm_plate_t/2}" rpy="0 0 ${q_yaw}"/>
     <axis xyz="0 0 1"/>
     <limit lower="${-servo_limit}" upper="${servo_limit}" effort="${servo_effort}" velocity="${servo_velocity}"/>
@@ -92,5 +107,5 @@
     <parent link="arm_turret"/>
     <child link="upper_arm"/>
-    <origin xyz="0 0 ${arm_l1}"/>
+    <origin xyz="0 0 ${arm_l1}" rpy="0 ${q_shoulder} 0"/>
     <axis xyz="0 1 0"/>
     <limit lower="${-servo_limit}" upper="${servo_limit}" effort="${servo_effort}" velocity="${servo_velocity}"/>
@@ -101,5 +116,5 @@
     <parent link="upper_arm"/>
     <child link="forearm"/>
-    <origin xyz="0 0 ${arm_l2}"/>
+    <origin xyz="0 0 ${arm_l2}" rpy="0 ${q_elbow} 0"/>
     <axis xyz="0 1 0"/>
     <limit lower="${-servo_limit}" upper="${servo_limit}" effort="${servo_effort}" velocity="${servo_velocity}"/>
@@ -110,5 +125,5 @@
     <parent link="forearm"/>
     <child link="wrist"/>
-    <origin xyz="0 0 ${arm_l3}"/>
+    <origin xyz="0 0 ${arm_l3}" rpy="0 ${q_wrist} 0"/>
     <axis xyz="0 1 0"/>
     <limit lower="${-servo_limit}" upper="${servo_limit}" effort="${servo_effort}" velocity="${servo_velocity}"/>
@@ -116,5 +131,5 @@
   <link name="wrist">
     <visual><origin xyz="0 0 ${wrist_roll_z/2}"/><geometry><box size="${link_w} ${link_w} ${wrist_roll_z}"/></geometry><material name="petg_blue"/></visual>
-    <collision><origin xyz="0 0 ${wrist_roll_z/2}"/><geometry><box size="${servo_x} ${servo_y} ${wrist_roll_z+servo_z}"/></geometry></collision>
+    <collision><origin xyz="0 0 ${wrist_roll_z/2}"/><geometry><box size="${servo_x} ${arm_scan_w} ${wrist_roll_z+servo_z}"/></geometry></collision>
     <inertial><origin xyz="0 0 ${wrist_roll_z/2}"/><mass value="0.1"/><xacro:box_inertia m="0.1" x="${servo_x}" y="${servo_y}" z="${wrist_roll_z}"/></inertial>
   </link>
@@ -130,5 +145,5 @@
     <parent link="wrist"/>
     <child link="nozzle"/>
-    <origin xyz="0 0 ${wrist_roll_z}"/>
+    <origin xyz="0 0 ${wrist_roll_z}" rpy="0 0 ${q_roll}"/>
     <axis xyz="0 0 1"/>
     <limit lower="${-servo_limit}" upper="${servo_limit}" effort="${servo_effort}" velocity="${servo_velocity}"/>

File: description/weedbot_properties.xacro (robot description, xacro)
@@ -63,5 +63,6 @@
   <xacro:property name="tank_w"    value="0.239"/>
   <xacro:property name="tank_z0"   value="0.2305"/>
-  <xacro:property name="tank_z1"   value="0.3544"/>
+  <xacro:property name="tank_z1"   value="0.3474"/>   <!-- tank top (v19) = puck bottom; the filler cap reaches 0.3604
+                                                          (not modelled: position not given, below the scan plane) -->
   <xacro:property name="sump_x0"   value="0.203"/>
   <xacro:property name="sump_x1"   value="0.271"/>
@@ -71,9 +72,10 @@
   <!-- robotic arm: 4 x MG996R pitch/yaw (40.7 x 19.7 x 42.9 mm, 180 deg) + wrist roll -->
   <xacro:property name="arm_x"          value="-0.0066"/>    <!-- base yaw axis (v19: arm base on the top cover) -->
-  <xacro:property name="arm_base_z"     value="0.2305"/>     <!-- underside of the arm base plate (= top of the top frame) -->
-  <xacro:property name="arm_plate_t"    value="0.0061"/>     <!-- plate top = yaw joint = top of the cover, 0.2366 -->
+  <xacro:property name="arm_base_z"     value="0.2305"/>     <!-- underside of the bearing plate set into the cover (= top of the top frame) -->
+  <xacro:property name="arm_plate_t"    value="0.0061"/>     <!-- plate top = yaw joint = top of the cover 0.2366 = underside of
+                                                                  the turning arm base, which sits on the cover -->
   <xacro:property name="arm_plate_r"    value="0.060"/>
   <xacro:property name="arm_yaw_servo_dx" value="-0.0224"/>  <!-- yaw servo under the plate, behind the axis (drives a gear) -->
-  <xacro:property name="arm_l1"         value="0.0707"/>     <!-- base plate to shoulder axis -->
+  <xacro:property name="arm_l1"         value="0.07065"/>    <!-- arm base underside (yaw joint) to shoulder axis -->
   <xacro:property name="arm_l2"         value="0.100"/>      <!-- shoulder axis to elbow axis -->
   <xacro:property name="arm_l3"         value="0.100"/>      <!-- elbow axis to wrist pitch axis -->
@@ -85,4 +87,16 @@
   <xacro:property name="servo_velocity" value="5.0"/>       <!-- rad/s (0.17 s / 60 deg) -->
   <xacro:property name="link_w"         value="0.020"/>
+  <xacro:property name="arm_scan_w"     value="0.078"/>     <!-- width (y) of the wrist COLLISION box: CAD v19 says the parked arm
+                                                                 blocks ~32 deg behind the LD06; the wrist (servo + brackets) is the
+                                                                 nearest arm part in the scan plane, 0.136 m away: 2 x 0.136 x tan 16 deg.
+                                                                 Makes the sim scan match; visuals keep the plain servo boxes. -->
+  <!-- parked pose (CAD v19): upper arm straight up, forearm pointing forward (horizontal), last link
+       pointing down: wrist axis x +0.0934 at 0.40725, nozzle tip at 0.27625. The sim fixes the arm in
+       this pose; config/arm_joint_state_stub.yaml publishes the same angles for the real robot. -->
+  <xacro:property name="arm_park_yaw"      value="0.0"/>
+  <xacro:property name="arm_park_shoulder" value="0.0"/>
+  <xacro:property name="arm_park_elbow"    value="${pi/2}"/>
+  <xacro:property name="arm_park_wrist"    value="${pi/2}"/>
+  <xacro:property name="arm_park_roll"     value="0.0"/>
   <!-- phone mount (printed cradle + wedge bracket) on the deck at the front. May move to the nose. -->
   <xacro:property name="phone_bracket_x" value="0.1882"/>   <!-- rear edge of the WedgeBracket base from the rear axle -->
