Commit message: URDF: v21 CAD - front is the drive end, LD06 on the tank, arm on the body, phone mount
- weedbot_properties.xacro: CAD v21 values; x now points to the drive-wheel end (arm, phone),
  caster at x -0.419 behind, tank/sump/LD06/electronics at the back, arm_x 0.0066,
  arm_plate_r 0.0715 + 0.023 base housing, arm_l1 0.0707, wrist_roll_z renamed arm_roll_d,
  tank top 0.3544, lidar_yaw (0 = LD06 0 deg mark toward the arm), new phone mount numbers.
- weedbot_body.xacro: caster bracket behind the frame, top cover from the tank forward,
  phone_shelf / phone_bracket / tilted phone_cradle + phone_body; camera frames at phone_xyz.
- weedbot_arm.xacro: round base housing on the turret; the upper arm's collision box is widened
  (arm_scan_w 0.087) so the sim shows the CAD's +-10 deg blind sector straight ahead.
- ros2_control.xacro: real robot drive flipped without rewiring or firmware changes: wheel names
  swapped and enc_counts_per_rev -3436 (inverts motor commands and encoder signs). Needs the
  wheels-off-the-ground check on the robot.
- Nav2 footprint (both costmaps) for the new outline; safety.yaml StopBand / SlowCorridor ahead
  of the phone mount, stop_zone and scan_self_filter box (x -0.53..0.18) mirrored.
- CLAUDE.md: v21 layout and heights, drive direction check, blind-wedge safety findings.

Sim (domain 42): 20 deg self-hit sector straight ahead, all NaN after the filter; teleop forward
moves toward the arm, left turns CCW. A person straight ahead is invisible beyond x ~0.9 and the
robot drove into an 8 cm post on the centre line: the wedge needs a fix before autonomous driving.

Co-Authored-By: Claude Opus 5.5 <noreply@anthropic.com>

File: description/imu.xacro (robot description, xacro)
@@ -3,5 +3,8 @@
   <!-- MPU6050 position measured from the point between the drive wheels, in metres.
        Board flat, printed X arrow pointing forward, Y pointing left.
-       If it is rotated, change the rpy here OR the axis_signs in imu_ekf.launch.py, not both. -->
+       If it is rotated, change the rpy here OR the axis_signs in imu_ekf.launch.py, not both.
+       Forward = the drive-wheel end since CAD v21 (it was the caster end): an X arrow pointing at the
+       caster is a 180 deg rotation (rpy 0 0 pi). The EKF only uses the z gyro, which does not change.
+       Position: MEASURE. -->
   <xacro:property name="imu_x" value="0.05"/>
   <xacro:property name="imu_y" value="0.00"/>

File: description/lidar_sim.xacro (robot description, xacro)
@@ -20,11 +20,10 @@
         </scan>
         <range>
-          <!-- 0.14 (v19, LD06 on the tank): every ray must START outside the tank's outline seen from
-               above (farthest tank corner 0.130 m from the laser). With 0.05 the backward rays started
-               above the tank top (2.4 cm below the scan plane) and Gazebo's ray-box test reported
-               flickering false hits at the tank's rear edge (0.052 m) whenever the robot pitched a
-               hair nose-up. Everything within 0.14 m is inside scan_self_filter's box anyway. The
-               parked arm still gives the real ~32 deg sector behind; its wrist's near face (0.136 m)
-               is just inside 0.14, so the sim reports the far face (0.176 m): filtered either way. -->
+          <!-- 0.14 (LD06 on the tank): every ray must START outside the tank's outline seen from
+               above (farthest tank corner 0.130 m from the laser). With 0.05 the rays over the tank
+               started above the tank top (2.4 cm below the scan plane) and Gazebo's ray-box test
+               reported flickering false hits at the tank's edge (0.052 m) whenever the robot pitched
+               a hair. Everything within 0.14 m is inside scan_self_filter's box anyway. The parked
+               arm in front of the LD06 gives the real ~+-10 deg sector straight ahead. -->
           <min>0.14</min>
           <max>12</max>

File: description/robot.urdf.xacro (robot description, xacro)
@@ -1,6 +1,7 @@
 <?xml version="1.0"?>
-<!-- WeedBot (rebuilt 2026-10): rear differential drive + front stem caster, spray tank with the LD06
-     on top, sprayer arm on the top cover, phone mount. All measurements: weedbot_properties.xacro (MEASURE markers).
-     base_link = on the ground under the centre of the rear axle.
+<!-- WeedBot (CAD v21): FRONT = the drive-wheel end, with the sprayer arm on the top cover and the
+     phone mount on a shelf on the front; stem caster at the back, spray tank at the back with the LD06
+     on top. All measurements: weedbot_properties.xacro (MEASURE markers).
+     base_link = on the ground under the centre of the drive axle.
      Old files kept on disk but no longer included: robot_core.xacro, lidar.xacro, camera.xacro,
      phone_mount.xacro (the body defines phone_mount -> phone_optical -> phone_link itself). -->

File: description/ros2_control.xacro (robot description, xacro)
@@ -3,13 +3,23 @@
     <xacro:unless value="$(arg sim_mode)">
         <ros2_control name="RealRobot" type="system">
+            <!-- CAD v21: the FRONT is now the drive-wheel end (it was the caster end). Nothing was
+                 rewired, so each motor is now on the other side of the robot and "its" forward is
+                 now backward. Both are fixed here, firmware unchanged:
+                 - left/right_wheel_name SWAPPED: the Arduino's LEFT channel (first number of
+                   "m L R" and of "e") drives the wheel that is now on the RIGHT (y -0.088);
+                 - enc_counts_per_rev NEGATIVE: diffdrive_arduino uses rads_per_count =
+                   2*pi/enc_counts_per_rev for the motor command AND the encoder angle, so the
+                   minus sign inverts both motor directions and both encoder signs.
+                 Result: positive left/right_wheel_joint velocity drives toward the arm end.
+                 Check with the wheels off the ground (CLAUDE.md "Drive direction check"). -->
             <hardware>
                 <plugin>diffdrive_arduino/DiffDriveArduinoHardware</plugin>
-                <param name="left_wheel_name">left_wheel_joint</param>
-                <param name="right_wheel_name">right_wheel_joint</param>
+                <param name="left_wheel_name">right_wheel_joint</param>
+                <param name="right_wheel_name">left_wheel_joint</param>
                 <param name="loop_rate">30</param>
                 <param name="device">/dev/ttyACM0</param>
                 <param name="baud_rate">57600</param>
                 <param name="timeout_ms">5000</param>
-                <param name="enc_counts_per_rev">3436</param>
+                <param name="enc_counts_per_rev">-3436</param>
             </hardware>
             <joint name="left_wheel_joint">

File: description/weedbot_arm.xacro (robot description, xacro)
@@ -1,15 +1,17 @@
 <?xml version="1.0"?>
 <!--
-  Sprayer arm on the top cover (rear of the robot, CAD v19): 4 x MG996R + a wrist roll.
-    arm_base_yaw   : servo 1, hangs under the base plate behind the axis and turns the arm through
-                     a gear, about the vertical axis at arm_x (yaw range: MEASURE)
+  Sprayer arm on the top cover at the FRONT of the robot (over the drive wheels, CAD v21):
+  4 x MG996R + a wrist roll.
+    arm_base_yaw   : servo 1, hangs under the base plate in front of the axis and turns the arm (and
+                     its round base housing) through a gear, about the vertical axis at arm_x
+                     (yaw range: MEASURE)
     shoulder_pitch : servo 2
     elbow_pitch    : servo 3
     wrist_pitch    : servo 4
-    wrist_roll     : servo 5, wrist_roll_z along the last link, turns the nozzle about the link
+    wrist_roll     : servo 5, arm_roll_d along the last link, turns the nozzle about the link
                      (link spray_tip = where the spray leaves)
-  Zero position = arm pointing straight up. Positive pitch tilts forward.
+  Zero position = arm pointing straight up. Positive pitch tilts forward (toward the phone).
   Each joint: -90..+90 deg (the servo's 180 deg travel centred). Link lengths (axis to axis) are in
-  weedbot_properties.xacro (arm_l1..l4, wrist_roll_z, CAD v17). Masses: MEASURE.
+  weedbot_properties.xacro (arm_l1..l4, arm_roll_d, CAD v21). Masses: MEASURE.
   In RViz, move it with joint_state_publisher_gui; on the robot the servo driver publishes the same
   joint names on /joint_states.
@@ -47,6 +49,7 @@
     </visual>
   </xacro:macro>
-  <!-- arm link: a bar along +z of length L, with the next servo at its end -->
-  <xacro:macro name="arm_link" params="name length mass">
+  <!-- arm link: a bar along +z of length L, with the next servo at its end. scan_w = width (y) of the
+       collision box (wider than the bar only where the LD06 sees the arm, see arm_scan_w) -->
+  <xacro:macro name="arm_link" params="name length mass scan_w:=${link_w}">
     <link name="${name}">
       <visual>
@@ -57,5 +60,5 @@
       <collision>
         <origin xyz="0 0 ${length/2}"/>
-        <geometry><box size="${link_w} ${link_w} ${length}"/></geometry>
+        <geometry><box size="${link_w} ${scan_w} ${length}"/></geometry>
       </collision>
       <inertial>
@@ -77,6 +80,6 @@
     <inertial><mass value="0.15"/><xacro:cyl_inertia m="0.15" r="${arm_plate_r}" h="${arm_plate_t}"/></inertial>
   </link>
-  <!-- yaw servo (servo 1) under the plate (inside the body), arm_yaw_servo_dx behind the axis, shaft
-       up into the gear -->
+  <!-- yaw servo (servo 1) under the plate (inside the body), arm_yaw_servo_dx in front of the axis,
+       shaft up into the gear -->
   <joint name="arm_yaw_servo_joint" type="fixed">
     <parent link="arm_base"/>
@@ -93,12 +96,14 @@
     <limit lower="${-servo_limit}" upper="${servo_limit}" effort="${servo_effort}" velocity="${servo_velocity}"/>
   </joint>
+  <!-- turning part: round base housing on the cover + the post up to the shoulder -->
   <link name="arm_turret">
     <visual><origin xyz="0 0 ${arm_l1/2}"/><geometry><box size="${link_w} ${link_w} ${arm_l1}"/></geometry><material name="petg_blue"/></visual>
+    <visual><origin xyz="0 0 ${arm_housing_h/2}"/><geometry><cylinder radius="${arm_plate_r}" length="${arm_housing_h}"/></geometry><material name="petg_blue"/></visual>
+    <collision><origin xyz="0 0 ${arm_housing_h/2}"/><geometry><cylinder radius="${arm_plate_r}" length="${arm_housing_h}"/></geometry></collision>
     <inertial><origin xyz="0 0 ${arm_l1/2}"/><mass value="0.09"/><xacro:box_inertia m="0.09" x="${servo_x}" y="${servo_y}" z="${arm_l1}"/></inertial>
   </link>
-  <!-- turret disc on the plate and servo 2 (shoulder) body at the top -->
+  <!-- servo 2 (shoulder) body at the top of the post -->
   <joint name="turret_servo_joint" type="fixed"><parent link="arm_turret"/><child link="turret_servo"/><origin xyz="0 0 0"/></joint>
   <link name="turret_servo">
-    <visual><origin xyz="0 0 0.004"/><geometry><cylinder radius="0.030" length="0.008"/></geometry><material name="servo"/></visual>
     <xacro:servo_visual xyz="0 0 ${arm_l1-servo_z/2+0.005}" rpy="0 0 0"/>
   </link>
@@ -111,5 +116,5 @@
     <limit lower="${-servo_limit}" upper="${servo_limit}" effort="${servo_effort}" velocity="${servo_velocity}"/>
   </joint>
-  <xacro:arm_link name="upper_arm" length="${arm_l2}" mass="0.08"/>
+  <xacro:arm_link name="upper_arm" length="${arm_l2}" mass="0.08" scan_w="${arm_scan_w}"/>
   <!-- servo 3: elbow -->
   <joint name="elbow_pitch" type="${arm_joint_type}">
@@ -130,7 +135,7 @@
   </joint>
   <link name="wrist">
-    <visual><origin xyz="0 0 ${wrist_roll_z/2}"/><geometry><box size="${link_w} ${link_w} ${wrist_roll_z}"/></geometry><material name="petg_blue"/></visual>
-    <collision><origin xyz="0 0 ${wrist_roll_z/2}"/><geometry><box size="${servo_x} ${arm_scan_w} ${wrist_roll_z+servo_z}"/></geometry></collision>
-    <inertial><origin xyz="0 0 ${wrist_roll_z/2}"/><mass value="0.1"/><xacro:box_inertia m="0.1" x="${servo_x}" y="${servo_y}" z="${wrist_roll_z}"/></inertial>
+    <visual><origin xyz="0 0 ${arm_roll_d/2}"/><geometry><box size="${link_w} ${link_w} ${arm_roll_d}"/></geometry><material name="petg_blue"/></visual>
+    <collision><origin xyz="0 0 ${arm_roll_d/2}"/><geometry><box size="${servo_x} ${servo_y} ${arm_roll_d+servo_z}"/></geometry></collision>
+    <inertial><origin xyz="0 0 ${arm_roll_d/2}"/><mass value="0.1"/><xacro:box_inertia m="0.1" x="${servo_x}" y="${servo_y}" z="${arm_roll_d}"/></inertial>
   </link>
   <!-- servo 4 body at the wrist pitch axis and servo 5 (wrist roll) body, shaft along the link at the
@@ -139,5 +144,5 @@
   <link name="wrist_servos">
     <xacro:servo_visual xyz="0 0 0" rpy="0 0 0"/>
-    <visual><origin xyz="0 0 ${wrist_roll_z-servo_x/2}"/><geometry><box size="${servo_y} ${servo_z} ${servo_x}"/></geometry><material name="servo"/></visual>
+    <visual><origin xyz="0 0 ${arm_roll_d-servo_x/2}"/><geometry><box size="${servo_y} ${servo_z} ${servo_x}"/></geometry><material name="servo"/></visual>
   </link>
   <!-- servo 5: wrist roll, turns the nozzle about the link axis -->
@@ -145,12 +150,12 @@
     <parent link="wrist"/>
     <child link="nozzle"/>
-    <origin xyz="0 0 ${wrist_roll_z}" rpy="0 0 ${q_roll}"/>
+    <origin xyz="0 0 ${arm_roll_d}" rpy="0 0 ${q_roll}"/>
     <axis xyz="0 0 1"/>
     <limit lower="${-servo_limit}" upper="${servo_limit}" effort="${servo_effort}" velocity="${servo_velocity}"/>
   </joint>
   <link name="nozzle">
-    <visual><origin xyz="0 0 ${(arm_l4-wrist_roll_z)/2}"/><geometry><cylinder radius="0.006" length="${arm_l4-wrist_roll_z}"/></geometry><material name="alu"/></visual>
-    <collision><origin xyz="0 0 ${(arm_l4-wrist_roll_z)/2}"/><geometry><cylinder radius="0.006" length="${arm_l4-wrist_roll_z}"/></geometry></collision>
-    <inertial><origin xyz="0 0 ${(arm_l4-wrist_roll_z)/2}"/><mass value="0.02"/><xacro:cyl_inertia m="0.02" r="0.006" h="${arm_l4-wrist_roll_z}"/></inertial>
+    <visual><origin xyz="0 0 ${(arm_l4-arm_roll_d)/2}"/><geometry><cylinder radius="0.006" length="${arm_l4-arm_roll_d}"/></geometry><material name="alu"/></visual>
+    <collision><origin xyz="0 0 ${(arm_l4-arm_roll_d)/2}"/><geometry><cylinder radius="0.006" length="${arm_l4-arm_roll_d}"/></geometry></collision>
+    <inertial><origin xyz="0 0 ${(arm_l4-arm_roll_d)/2}"/><mass value="0.02"/><xacro:cyl_inertia m="0.02" r="0.006" h="${arm_l4-arm_roll_d}"/></inertial>
   </link>
   <!-- where the spray comes out, z pointing along the nozzle -->
@@ -158,5 +163,5 @@
     <parent link="nozzle"/>
     <child link="spray_tip"/>
-    <origin xyz="0 0 ${arm_l4-wrist_roll_z}"/>
+    <origin xyz="0 0 ${arm_l4-arm_roll_d}"/>
   </joint>
   <link name="spray_tip">
